File: trackduino micro/trackduino1309111914.brd (EAGLE design)
At the start: 52.6 x 22.3 mm, 35 parts, among them IC1 74AHC1G125DBV, IC2 74AHC1G125DBV, IC3 74AHC1G125DBV, U1 ATMEGA168

Commit message: swapped crystal for smaller resonator
Parts:
- removed C6, C7: (no value), SparkFun-Capacitors:0805
- removed Q1: (no value), crystal:CTS406
- added Y1: 16MHZ, SparkFun-FreqCtrl:RESONATOR-SMD
Connections:
- net GND: now also Y1.2; no longer C6.1, C7.1
- net N$14: now also U1.8, Y1.3; no longer C6.2, Q1.3, U1.7
- net N$26: now also U1.7, Y1.1; no longer C7.2, Q1.1, U1.8
Routing:
- net N$14: track 14.4 -> 2.40 mm, vias 1 -> 0
- net N$26: track 6.15 -> 1.17 mm, vias 1 -> 0
- net GND: track 178.5 -> 180.2 mm
Changed lines of the file:
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@@
 <attribute name="PROD_ID" value="SWCH-08247" x="95.631" y="60.1218" size="1.778" layer="27" display="off"/>
 </element>
-<element name="Q1" library="crystal" package="CTS406" value="" x="63.8155375" y="68.249578125" rot="R135">
-<attribute name="OC_NEWARK" value="unknown" x="63.8155375" y="68.249578125" size="1.778" layer="27" rot="R135" display="off"/>
-<attribute name="MPN" value="" x="63.8155375" y="68.249578125" size="1.778" layer="27" rot="R135" display="off"/>
-<attribute name="MF" value="" x="63.8155375" y="68.249578125" size="1.778" layer="27" rot="R135" display="off"/>
-<attribute name="OC_FARNELL" value="unknown" x="63.8155375" y="68.249578125" size="1.778" layer="27" rot="R135" display="off"/>
-</element>
-<element name="C6" library="SparkFun-Capacitors" package="0805" value="" x="60.449446875" y="67.5193625" rot="R135"/>
-<element name="C7" library="SparkFun-Capacitors" package="0805" value="" x="68.1179125" y="67.846484375" rot="R135"/>
 <element name="FRAME1" library="SparkFun-Aesthetics" package="CREATIVE_COMMONS" value="FRAME-LETTER" x="65.7606" y="49.3522"/>
 <element name="LED4" library="adafruit" package="CHIP-LED0805" value="" x="49.0474" y="69.1896" rot="MR270"/>
 <element name="R6" library="SparkFun-Resistors" package="0805" value="" x="52.5272" y="69.1896" rot="MR180"/>
+<element name="Y1" library="SparkFun-FreqCtrl" package="RESONATOR-SMD" value="16MHZ" x="69.510028125" y="70.91935" rot="MR225">
+<attribute name="PROD_ID" value="XTAL-08900" x="69.510028125" y="70.91935" size="1.778" layer="28" rot="MR225" display="off"/>
+</element>
 </elements>
 <signals>
@@
 <wire x1="85.2424" y1="60.0202" x2="82.7278" y2="60.0202" width="0.4064" layer="1"/>
 <wire x1="82.7278" y1="60.0202" x2="81.3054" y2="58.5978" width="0.4064" layer="1"/>
-<wire x1="96.6978" y1="64.1604" x2="96.9772" y2="64.262" width="0.4064" layer="1"/>
 <wire x1="77.1652" y1="64.1968" x2="77.5146" y2="64.1968" width="0.4064" layer="16"/>
 <wire x1="77.5146" y1="64.1968" x2="78.871" y2="62.8404" width="0.4064" layer="16"/>
@@
 <wire x1="73.66" y1="71.1708" x2="73.66" y2="72.0804" width="0.4064" layer="16"/>
 <wire x1="73.66" y1="72.0804" x2="72.7256" y2="73.0148" width="0.4064" layer="16"/>
-<wire x1="72.7256" y1="73.0148" x2="72.0446" y2="73.0148" width="0.4064" layer="16"/>
+<wire x1="72.7256" y1="73.0148" x2="72.2122" y2="73.0148" width="0.4064" layer="16"/>
+<wire x1="72.2122" y1="73.0148" x2="72.0446" y2="73.0148" width="0.4064" layer="16"/>
 <wire x1="72.0446" y1="73.0148" x2="71.7804" y2="73.279" width="0.4064" layer="16"/>
 <wire x1="71.7804" y1="73.279" x2="71.7804" y2="74.5592" width="0.4064" layer="16"/>
@@
 <vertex x="46.7106" y="57.023"/>
 </polygon>
-<contactref element="C6" pad="1"/>
-<contactref element="C7" pad="1"/>
-<wire x1="68.75430625" y1="67.2100875" x2="69.15901875" y2="67.6148" width="0.4064" layer="1"/>
-<wire x1="69.15901875" y1="67.6148" x2="70.3326" y2="67.6148" width="0.4064" layer="1"/>
-<wire x1="61.085840625" y1="66.882965625" x2="61.8744" y2="66.09440625" width="0.4064" layer="1"/>
 <wire x1="61.8744" y1="66.09440625" x2="61.8744" y2="66.0908" width="0.4064" layer="1"/>
 <via x="61.8744" y="66.0908" extent="1-16" drill="0.6" shape="square"/>
@@
 <contactref element="LED4" pad="C"/>
 <wire x1="47.9974" y1="70.7644" x2="47.9974" y2="69.1896" width="0.4064" layer="16"/>
-<wire x1="96.6978" y1="64.1604" x2="98.425" y2="58.2168" width="0" layer="19" extent="1-1"/>
+<contactref element="Y1" pad="2"/>
+<wire x1="68.791609375" y1="70.200928125" x2="70.67588125" y2="72.0852" width="0.4064" layer="16"/>
+<wire x1="70.67588125" y1="72.0852" x2="71.7296" y2="72.0852" width="0.4064" layer="16"/>
+<wire x1="71.7296" y1="72.0852" x2="72.2122" y2="72.5678" width="0.4064" layer="16"/>
+<wire x1="72.2122" y1="72.5678" x2="72.2122" y2="73.0148" width="0.4064" layer="16"/>
+<wire x1="96.9772" y1="64.262" x2="98.425" y2="58.2168" width="0" layer="19" extent="1-1"/>
 <wire x1="96.9772" y1="64.262" x2="96.9772" y2="64.262" width="0" layer="19" extent="1-16"/>
 <wire x1="56.515" y1="65.9384" x2="59.19123125" y2="66.233915625" width="0" layer="19" extent="16-16"/>
@@
 <wire x1="72.8218" y1="66.9544" x2="73.5534" y2="66.9544" width="0.4064" layer="16"/>
 <wire x1="73.5534" y1="66.9544" x2="74.7116" y2="68.1126" width="0.4064" layer="16"/>
-<wire x1="69.3928" y1="74.19060625" x2="70.5612" y2="73.02220625" width="0.4064" layer="16"/>
-<wire x1="70.5612" y1="73.02220625" x2="70.5612" y2="72.0598" width="0.4064" layer="16"/>
-<via x="70.5612" y="72.0598" extent="1-16" drill="0.6" shape="square"/>
-<wire x1="70.5612" y1="72.0598" x2="71.247" y2="71.374" width="0.4064" layer="1"/>
-<wire x1="71.247" y1="71.374" x2="77.0128" y2="71.374" width="0.4064" layer="1"/>
+<wire x1="69.3928" y1="74.19060625" x2="69.4944" y2="74.13980625" width="0.4064" layer="16"/>
+<wire x1="69.4944" y1="74.13980625" x2="70.3834" y2="73.0758" width="0.4064" layer="16"/>
+<via x="70.3834" y="73.0758" extent="1-16" drill="0.6" shape="square"/>
+<wire x1="70.3834" y1="73.0758" x2="71.7296" y2="71.4248" width="0.4064" layer="1"/>
+<wire x1="71.7296" y1="71.4248" x2="77.0128" y2="71.374" width="0.4064" layer="1"/>
 <via x="77.0128" y="71.374" extent="1-16" drill="0.6" shape="square"/>
 <wire x1="77.0128" y1="71.374" x2="77.343" y2="71.9328" width="0.4064" layer="16"/>
@@
 <wire x1="64.366203125" y1="74.803" x2="65.2272" y2="74.6506" width="0.4064" layer="16"/>
 <via x="65.2272" y="74.6506" extent="1-16" drill="0.6" shape="square"/>
-<wire x1="65.2272" y1="74.6506" x2="69.977" y2="69.8754" width="0.4064" layer="1"/>
-<wire x1="69.977" y1="69.8754" x2="70.7644" y2="69.1388" width="0.4064" layer="1"/>
-<via x="70.7644" y="69.1388" extent="1-16" drill="0.6" shape="square"/>
-<wire x1="70.7644" y1="69.1388" x2="70.8914" y2="69.0118" width="0.4064" layer="16"/>
-<wire x1="70.8914" y1="69.0118" x2="72.7002" y2="69.0626" width="0.4064" layer="16"/>
+<wire x1="65.2272" y1="74.6506" x2="70.739" y2="69.1388" width="0.4064" layer="1"/>
+<wire x1="70.739" y1="69.1388" x2="71.0438" y2="69.1388" width="0.4064" layer="1"/>
+<via x="71.0438" y="69.1388" extent="1-16" drill="0.6" shape="square"/>
+<wire x1="71.0438" y1="69.1388" x2="71.4756" y2="69.0626" width="0.4064" layer="16"/>
+<wire x1="71.4756" y1="69.0626" x2="72.7002" y2="69.0626" width="0.4064" layer="16"/>
 </signal>
 <signal name="TX">
@@
 <signal name="N$11">
 </signal>
-<signal name="N$14">
-<contactref element="U1" pad="7"/>
-<contactref element="Q1" pad="3"/>
-<wire x1="66.958940625" y1="70.6075125" x2="66.049028125" y2="69.6976" width="0.4064" layer="16"/>
-<wire x1="66.049028125" y1="69.6976" x2="65.7098" y2="69.6976" width="0.4064" layer="16"/>
-<via x="65.7098" y="69.6976" extent="1-16" drill="0.6" shape="square"/>
-<wire x1="65.7098" y1="69.6976" x2="62.4586" y2="72.9488" width="0.4064" layer="1"/>
-<wire x1="62.4586" y1="72.9488" x2="61.2648" y2="72.9488" width="0.4064" layer="1"/>
-<wire x1="61.2648" y1="72.9488" x2="60.071" y2="71.755" width="0.4064" layer="1"/>
-<wire x1="60.071" y1="71.755" x2="60.071" y2="70.2818" width="0.4064" layer="1"/>
-<wire x1="60.071" y1="70.2818" x2="61.396115625" y2="68.956684375" width="0.4064" layer="1"/>
-<wire x1="61.396115625" y1="68.956684375" x2="61.411371875" y2="68.956684375" width="0.4064" layer="1"/>
-<contactref element="C6" pad="2"/>
-<contactref element="C6" pad="2"/>
-<wire x1="59.81305" y1="68.15575625" x2="60.613978125" y2="68.956684375" width="0.4064" layer="1"/>
-<wire x1="60.613978125" y1="68.956684375" x2="61.411371875" y2="68.956684375" width="0.4064" layer="1"/>
-</signal>
-<signal name="N$26">
-<contactref element="U1" pad="8"/>
-<contactref element="Q1" pad="1"/>
-<wire x1="66.2197" y1="67.54246875" x2="68.14623125" y2="69.469" width="0.4064" layer="1"/>
-<wire x1="68.14623125" y1="69.469" x2="68.6054" y2="69.469" width="0.4064" layer="1"/>
-<via x="68.6054" y="69.469" extent="1-16" drill="0.6" shape="square"/>
-<wire x1="68.6054" y1="69.469" x2="68.032575" y2="70.041825" width="0.4064" layer="16"/>
-<wire x1="68.032575" y1="70.041825" x2="67.524628125" y2="70.041825" width="0.4064" layer="16"/>
-<contactref element="C7" pad="2"/>
-<contactref element="C7" pad="2"/>
-<wire x1="66.2197" y1="67.54246875" x2="67.160109375" y2="68.482878125" width="0.4064" layer="1"/>
-<wire x1="67.160109375" y1="68.482878125" x2="67.481515625" y2="68.482878125" width="0.4064" layer="1"/>
-</signal>
 <signal name="N$27">
 <contactref element="LED4" pad="A"/>
@@
 <wire x1="61.8998" y1="73.5558" x2="61.453975" y2="74.001625" width="0.4064" layer="16"/>
 </signal>
+<signal name="N$14">
+<contactref element="U1" pad="8"/>
+<contactref element="Y1" pad="3"/>
+<wire x1="67.524628125" y1="70.041825" x2="68.214053125" y2="69.3524" width="0.4064" layer="16"/>
+<wire x1="68.214053125" y1="69.3524" x2="69.6401375" y2="69.3524" width="0.4064" layer="16"/>
+</signal>
+<signal name="N$26">
+<contactref element="U1" pad="7"/>
+<contactref element="Y1" pad="1"/>
+<wire x1="66.958940625" y1="70.6075125" x2="67.400884375" y2="71.04945625" width="0.4064" layer="16"/>
+<wire x1="67.400884375" y1="71.04945625" x2="67.94308125" y2="71.04945625" width="0.4064" layer="16"/>
+</signal>
 </signals>
