File: trackduino micro/trackduino micro.brd (EAGLE design)
At the start: 48.1 x 21.9 mm, 28 parts, among them IC2 74AHC1G125DBV, SW1 SPST_TACT-KMR2, U1 ATMEGA168MLF, Y1 16MHZ

Commit message: fixed some routing
Parts:
- moved R5 3.21 mm to (64.6, 75.6), turned to 180 degrees
Routing:
- net VCC: track 87.5 -> 85.2 mm
- net TXO: track 13.6 -> 12.8 mm
- net RXO: track 16.0 -> 15.3 mm
