File: trackduino micro/trackduino micro.brd (EAGLE design)
At the start: 48.1 x 21.9 mm, 28 parts, among them IC2 74AHC1G125DBV, SW1 SPST_TACT-KMR2, U1 ATMEGA168MLF, Y1 16MHZ

Commit message: capacitors do not fit underneath things
Parts:
- moved C1 1.22 mm to (92.9, 70.1), flipped to the top
Routing:
- net GND: track 145.6 -> 154.7 mm, vias 8 -> 9
- net 3V: vias 2 -> 3
Changed lines of the file:
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@@
 <element name="R1" library="SparkFun-Resistors" package="0805" value="" x="78.9178" y="70.0278" rot="MR270"/>
 <element name="LED1" library="adafruit" package="CHIP-LED0805" value="" x="78.9178" y="66.8274" rot="MR180"/>
-<element name="C1" library="SparkFun-Capacitors" package="0805" value="" x="92.837" y="71.2978" rot="MR90"/>
+<element name="C1" library="SparkFun-Capacitors" package="0805" value="" x="92.9386" y="70.0786" rot="R90"/>
 <element name="C2" library="SparkFun-Capacitors" package="0805" value="" x="52.8574" y="73.025" rot="MR270"/>
 <element name="C3" library="SparkFun-Capacitors" package="0805" value="" x="66.1924" y="66.9798" rot="MR315"/>
@@
 <wire x1="93.4974" y1="65.7352" x2="93.4974" y2="64.5306" width="0.4064" layer="16"/>
 <wire x1="93.4974" y1="64.5306" x2="93.4794" y2="64.5126" width="0.4064" layer="16"/>
-<wire x1="93.4794" y1="64.5126" x2="93.4794" y2="59.2288" width="0.4064" layer="16"/>
-<wire x1="93.4794" y1="59.2288" x2="93.7802" y2="58.928" width="0.4064" layer="16"/>
 <wire x1="93.7802" y1="58.928" x2="91.0302" y2="58.928" width="0.4064" layer="16"/>
 <wire x1="56.928" y1="78.651" x2="60.928" y2="78.651" width="0.4064" layer="16"/>
@@
 <wire x1="74.422" y1="76.4032" x2="75.3872" y2="77.3684" width="0.4064" layer="1"/>
 <wire x1="75.3872" y1="77.3684" x2="75.3872" y2="77.8764" width="0.4064" layer="1"/>
+<wire x1="93.4794" y1="64.5126" x2="93.4794" y2="59.2288" width="0.8128" layer="16"/>
+<wire x1="93.4794" y1="59.2288" x2="93.7802" y2="58.928" width="0.8128" layer="16"/>
+<wire x1="91.0302" y1="58.928" x2="91.3638" y2="59.2616" width="0.8128" layer="16"/>
+<wire x1="91.3638" y1="59.2616" x2="91.3638" y2="64.6176" width="0.8128" layer="16"/>
+<wire x1="93.218" y1="66.0146" x2="92.9386" y2="66.294" width="0.4064" layer="16"/>
+<wire x1="92.9386" y1="66.294" x2="92.9386" y2="67.6402" width="0.4064" layer="16"/>
+<via x="92.9386" y="67.6402" extent="1-16" drill="0.6" shape="square"/>
+<wire x1="92.9386" y1="67.6402" x2="92.9386" y2="69.1786" width="0.4064" layer="1"/>
 <wire x1="47.4894" y1="68.0212" x2="48.6918" y2="63.373" width="0" layer="19" extent="1-16"/>
 </signal>
@@
 <wire x1="51.054" y1="77.4192" x2="53.7522" y2="77.4192" width="0.4064" layer="16"/>
 <wire x1="53.7522" y1="77.4192" x2="53.7616" y2="77.4286" width="0.4064" layer="16"/>
-<wire x1="91.3294" y1="74.0126" x2="91.567" y2="73.775" width="0.4064" layer="16" curve="-90"/>
-<wire x1="91.567" y1="73.775" x2="91.567" y2="72.4916" width="0.4064" layer="16"/>
-<wire x1="91.567" y1="72.4916" x2="91.567" y2="72.4408" width="0.4064" layer="16"/>
-<wire x1="92.837" y1="72.1978" x2="91.8608" y2="72.1978" width="0.4064" layer="16"/>
-<wire x1="91.8608" y1="72.1978" x2="91.567" y2="72.4916" width="0.4064" layer="16"/>
 <wire x1="52.8574" y1="72.125" x2="55.234" y2="72.125" width="0.4064" layer="16"/>
 <wire x1="55.234" y1="72.125" x2="57.0484" y2="73.9394" width="0.4064" layer="16"/>
@@
 <wire x1="92.4306" y1="75.692" x2="92.4306" y2="74.5206" width="0.4064" layer="16"/>
 <wire x1="92.4306" y1="74.5206" x2="92.9386" y2="74.0126" width="0.4064" layer="16"/>
+<wire x1="92.9386" y1="70.9786" x2="92.9386" y2="72.1868" width="0.4064" layer="1"/>
+<via x="92.9386" y="72.1868" extent="1-16" drill="0.6" shape="square"/>
+<wire x1="92.9386" y1="72.1868" x2="92.9386" y2="74.0126" width="0.4064" layer="16"/>
 </signal>
 <signal name="N$1">

Commit message: more layout issues
Test board 1
Parts:
- moved LED4 0.97 mm to (48.5, 67.1)
- moved R6 0.94 mm to (52.1, 67.1)
- moved R4 0.58 mm to (52.1, 68.9)
- moved LED3 0.56 mm to (48.5, 68.9)
- moved C1 0.15 mm to (92.9, 69.9)
- moved C2 0.06 mm to (52.9, 73.1)
Connections:
- new net S$1: C2.1, U$3.3
- net GND: no longer C2.1, U$3.3
Routing:
- net GND: track 154.7 -> 150.3 mm, vias 9 -> 8
- net S$1: track 0.00 -> 2.41 mm
- net VCC: track 85.2 -> 87.5 mm, vias 3 -> 2
