File: trackduino micro/trackduino1309111914.sch (EAGLE design)
At the start: 28 parts, among them IC2 74AHC1G125DBV, SW1 SPST_TACT-KMR2, U1 ATMEGA168, Y1 16MHZ

Commit message: Revert 658c1f1..8864008
This rolls back to commit 658c1f11e5b9c3d0ac6cf8412ef3704af54d539a.
Parts:
- removed SW1: SPST_TACT-KMR2, adafruit:SPST_TACT-KMR2
- removed X1: (no value), adafruit:ANTENNA_U.FL
- added IC1, IC3: 74AHC1G125DBV, 74xx-little-us:74AHC1G125DBV
- added J$2: SMA_EDGE, SparkFun-Connectors:SMA_EDGE
- added JP4: M02PTH, SparkFun-Connectors:M02PTH
- added L1: (no value), SparkFun-Passives:INDUCTOR0805
- added R2: (no value), SparkFun-Resistors:RESISTOR0805-RES
- added S1: TAC_SWITCHSMD, SparkFun-Electromechanical:TAC_SWITCHSMD
- U$1: value UBLOX_MAX -> UBLOX_NEO-6; device Ava:UBLOX_MAX -> Ava:UBLOX_NEO-6
Connections:
- new net EN-5V: IC3A.O, U$2.EN
- new net N$4: R2.1, U$1.8_RESERVED, U$1.9_VCC_RF
- new net N$5: L1.1, R2.2
- new net TXD-5V: IC1A.O, U$2.TXD
- net 3V: now also U$1.23_VCC; no longer U$1.7_VCC_IO, U$1.8_VCC, U$1.9_V_RESET
- net D3: now also IC1A.I; no longer U$2.TXD
- net D4: now also IC3A.I; no longer U$2.EN
- net GND: now also IC1A.OE, IC3A.OE, J$2.GND@0, J$2.GND@1, J$2.GND@2, J$2.GND@3, S1.3, S1.4, U$1.13_GND, U$1.24_GND; no longer SW1.S, SW1.S1, U$1.1_GND, X1.GND@0, X1.GND@1
- net N$2: now also U$1.3_TIMEPULSE; no longer U$1.4_TIMEPULSE
- net N$6: now also J$2.SIGNAL, L1.2; no longer X1.SIGNAL
- net N$9: now also S1.1, S1.2; no longer SW1.P, SW1.P1
- net RX: now also JP4.1, U$1.20_TXD1; no longer U$1.3_RXD1
- net RXO: now also JP4.2; no longer IC2A.I
- net TX: now also IC2A.I, U$1.21_RXD1; no longer U$1.2_TXD1
- net TX-3V3: no longer JP3.2
- net TXO: now also JP3.2
Other:
- moved on the sheet: LED1, R1
