File: trackduino micro/pico test.sch (EAGLE design)
At the start: 29 parts, among them IC2 74AHC1G125DBV, SW1 SPST_TACT-KMR2, U1 ATMEGA168MLF, X2 SMA-SMD, Y1 16MHZ

Commit message: minor fixes to smallest boards
Connections:
- new net SCL: U1.PC5(ADC5/SCL)
- new net SDA: U1.PC4(ADC4/SDA)
- net 3V: now also R5.2
- net VCC: no longer R5.2
Changed lines of the file:
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@@
 <part name="SUPPLY9" library="SparkFun-Aesthetics" deviceset="VCC" device=""/>
 <part name="R5" library="SparkFun-Resistors" deviceset="RESISTOR" device="0805-RES"/>
-<part name="SUPPLY10" library="SparkFun-Aesthetics" deviceset="VCC" device=""/>
 <part name="C5" library="SparkFun-Capacitors" deviceset="CAP" device="0805"/>
 <part name="JP3" library="SparkFun-Connectors" deviceset="M02" device="PTH"/>
@@
 <instance part="SUPPLY9" gate="G$1" x="208.28" y="55.88" rot="R270"/>
 <instance part="R5" gate="G$1" x="33.02" y="86.36" rot="R90"/>
-<instance part="SUPPLY10" gate="G$1" x="33.02" y="91.44"/>
 <instance part="C5" gate="G$1" x="17.78" y="81.28" rot="R90"/>
 <instance part="JP3" gate="G$1" x="231.14" y="66.04"/>
@@
 </segment>
 <segment>
-<pinref part="R5" gate="G$1" pin="2"/>
-<pinref part="SUPPLY10" gate="G$1" pin="VCC"/>
-</segment>
-<segment>
 <pinref part="U1" gate="G$1" pin="AVCC"/>
 <pinref part="SUPPLY11" gate="G$1" pin="VCC"/>
@@
 <label x="170.18" y="60.96" size="1.778" layer="95" rot="R180"/>
 <junction x="170.18" y="63.5"/>
+</segment>
+<segment>
+<pinref part="R5" gate="G$1" pin="2"/>
+<wire x1="33.02" y1="91.44" x2="33.02" y2="93.98" width="0.1524" layer="91"/>
+<label x="33.02" y="93.98" size="1.778" layer="95"/>
 </segment>
 </net>
@@
 </segment>
 </net>
+<net name="SDA" class="0">
+<segment>
+<pinref part="U1" gate="G$1" pin="PC4(ADC4/SDA)"/>
+<wire x1="81.28" y1="71.12" x2="83.82" y2="71.12" width="0.1524" layer="91"/>
+<label x="83.82" y="71.12" size="1.778" layer="95"/>
+</segment>
+</net>
+<net name="SCL" class="0">
+<segment>
+<pinref part="U1" gate="G$1" pin="PC5(ADC5/SCL)"/>
+<wire x1="81.28" y1="68.58" x2="83.82" y2="68.58" width="0.1524" layer="91"/>
+<label x="83.82" y="68.58" size="1.778" layer="95"/>
+</segment>
+</net>
