File: trackduino micro/trackuino micro sensor.sch (EAGLE design)
At the start: 34 parts, among them IC2 74AHC1G125DBV, SW1 SPST_TACT-KMR2, U1 ATMEGA168MLF, Y1 16MHZ

Commit message: trackuino sensor cleanup
Parts:
- added U$6: V_REG_MIC2920, SparkFun-PowerIC:V_REG_MIC2920
- C6: value (none) -> 47pf
- L1: value (none) -> 27nh
- R2: value (none) -> 10ohm
- RX: value M02PTH -> RX
- TX: value M02PTH -> TX
- renumbered JP2 to FTDI, JP3 to TX, JP4 to RX, JP5 to SPI
Connections:
- removed net N$9: C5.2, R5.1, SW1.P, SW1.P1, U1.PC6(/RESET)
- new net 15V: JP1.2, U$6.IN
- new net N$7: C5.2, R5.1, U1.PC6(/RESET)
- net DTR: now also SW1.P, SW1.P1
- net GND: now also U$6.GND
- net VCC: now also U$6.OUT; no longer JP1.2
Other:
- moved on the sheet: C5
