File: trackduino micro/trackuino micro sensor.brd (EAGLE design)
At the start: 48.1 x 21.9 mm, 34 parts, among them IC2 74AHC1G125DBV, SW1 SPST_TACT-KMR2, U1 ATMEGA168MLF, Y1 16MHZ

Commit message: trackuino sensor cleanup
Parts:
- removed JP4: M02PTH, SparkFun-Connectors:1X02
- added RX: RX, SparkFun-Connectors:1X02
- added U$6: V_REG_MIC2920, SparkFun-PowerIC:SOT223
- C6: value (none) -> 47pf
- L1: value (none) -> 27nh
- R2: value (none) -> 10ohm
- TX: value M02PTH -> TX
- moved J$1 4.71 mm to (53.4, 58.7)
- moved Y1 0.30 mm to (73.5, 61.9)
- renumbered JP2 to FTDI, JP3 to TX, JP5 to SPI
Connections:
- removed net N$9: C5.2, R5.1, SW1.1, SW1.3, U1.29
- new net 15V: JP1.2, U$6.1
- new net N$7: C5.2, R5.1, U1.29
- net DTR: now also SW1.1, SW1.3
- net GND: now also U$6.2
- net RXO: now also RX.1; no longer JP4.1
- net TX: now also RX.2; no longer JP4.2
- net VCC: now also U$6.3; no longer JP1.2
Routing:
- net GND: track 121.8 -> 148.2 mm, vias 2 -> 3
- net 15V: track 0.00 -> 25.1 mm
- net N$9: track 20.9 -> 3.30 mm
- net N$7: track 0.00 -> 13.9 mm
- net N$1: track 0.00 -> 7.52 mm
- net DTR: track 2.95 -> 9.61 mm
- net VCC: track 75.0 -> 81.4 mm, vias 5 -> 6
Other:
- board size 48.1 x 21.9 mm -> 43.3 x 19.1 mm

Commit message: traccino micro sensor
Parts:
- moved L1 0.08 mm to (91.5, 61.7)
Routing:
- net N$9: track 3.30 -> 0.00 mm
- net GND: track 148.2 -> 151.0 mm
Changed lines of the file:
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@@
 <element name="X1" library="adafruit" package="U.FL" value="" x="92.4052" y="58.928" rot="MR90"/>
 <element name="SW1" library="adafruit" package="KMR2" value="SPST_TACT-KMR2" x="58.9026" y="75.0316" rot="MR180"/>
-<element name="L1" library="SparkFun-Passives" package="0805" value="27nh" x="91.4908" y="61.7728" rot="MR0"/>
+<element name="L1" library="SparkFun-Passives" package="0805" value="27nh" x="91.4908" y="61.6966" rot="MR0"/>
 <element name="R2" library="SparkFun-Resistors" package="0805" value="10ohm" x="87.0204" y="60.4012" rot="MR90"/>
 <element name="C6" library="SparkFun-Capacitors" package="0805" value="47pf" x="88.9" y="60.4012" rot="MR270"/>
@@
 <via x="80.645" y="65.0494" extent="1-16" drill="0.6" shape="square"/>
 <contactref element="U$6" pad="2"/>
+<wire x1="53.2892" y1="58.674" x2="56.5912" y2="58.674" width="1.27" layer="1"/>
+<wire x1="56.5658" y1="58.6486" x2="56.5912" y2="58.674" width="0" layer="19" extent="1-1"/>
 <wire x1="52.1884" y1="67.183" x2="53.3908" y2="63.754" width="0" layer="19" extent="1-16"/>
-<wire x1="72.9996" y1="62.2032" x2="72.9996" y2="62.394721875" width="0.3048" layer="1"/>
-<wire x1="72.9996" y1="62.394721875" x2="72.79173125" y2="62.602590625" width="0.3048" layer="1"/>
+<wire x1="72.9996" y1="62.2032" x2="72.79173125" y2="62.602590625" width="0" layer="19" extent="1-16"/>
 </signal>
 <signal name="VCC">
@@
 <contactref element="L1" pad="1"/>
 <wire x1="92.4294" y1="63.522" x2="92.4294" y2="61.8114" width="0.3048" layer="16"/>
-<wire x1="92.4294" y1="61.8114" x2="92.3908" y2="61.7728" width="0.3048" layer="16"/>
-<wire x1="92.3908" y1="61.7728" x2="92.3908" y2="60.4674" width="0.3048" layer="16"/>
+<wire x1="92.4294" y1="61.8114" x2="92.3908" y2="61.6966" width="0.3048" layer="16"/>
+<wire x1="92.3908" y1="61.6966" x2="92.3908" y2="60.4674" width="0.3048" layer="16"/>
 <wire x1="92.3908" y1="60.4674" x2="92.4052" y2="60.453" width="0.3048" layer="16"/>
 </signal>
@@
 <wire x1="83.2866" y1="75.4126" x2="83.2866" y2="74.295" width="0.3048" layer="16"/>
 <wire x1="83.2866" y1="74.295" x2="82.804" y2="73.8124" width="0.3048" layer="16"/>
-<wire x1="82.804" y1="73.8124" x2="76.6318" y2="73.8124" width="0.3048" layer="16"/>
-<via x="76.6318" y="73.8124" extent="1-16" drill="0.6" shape="square"/>
-<wire x1="76.6318" y1="73.8124" x2="74.168" y2="73.8124" width="0.3048" layer="1"/>
+<wire x1="82.804" y1="73.8124" x2="80.6958" y2="73.8124" width="0.3048" layer="16"/>
+<via x="80.6958" y="73.8124" extent="1-16" drill="0.6" shape="square"/>
+<wire x1="80.6958" y1="73.8124" x2="74.168" y2="73.8124" width="0.3048" layer="1"/>
 <wire x1="74.168" y1="73.8124" x2="73.8632" y2="74.0918" width="0.3048" layer="1"/>
 <wire x1="73.8632" y1="74.0918" x2="66.9036" y2="74.0918" width="0.3048" layer="1"/>
@@
 <wire x1="87.0204" y1="59.5012" x2="87.1" y2="59.5012" width="0.3048" layer="16"/>
 <wire x1="87.1" y1="59.5012" x2="88.9" y2="61.3012" width="0.3048" layer="16"/>
-<wire x1="88.9" y1="61.3012" x2="89.3716" y2="61.7728" width="0.3048" layer="16"/>
-<wire x1="89.3716" y1="61.7728" x2="90.5908" y2="61.7728" width="0.3048" layer="16"/>
+<wire x1="88.9" y1="61.3012" x2="89.2954" y2="61.6966" width="0.3048" layer="16"/>
+<wire x1="89.2954" y1="61.6966" x2="90.5908" y2="61.6966" width="0.3048" layer="16"/>
 </signal>
 <signal name="TX1">
@@
 <wire x1="71.247" y1="68.42964375" x2="70.596278125" y2="67.778921875" width="0.3048" layer="16"/>
 </signal>
-<signal name="N$9">
-<wire x1="53.2892" y1="58.674" x2="56.5912" y2="58.674" width="1.27" layer="1"/>
-</signal>
 </signals>
