File: Tracksoar/tracksoar chip breakout shield.brd (EAGLE design)
At the start: 43.7 x 19.6 mm, 15 parts

Commit message: replace headers
replaced 2.54mm headers on all production boards with 2mm headers to
resolve daughter board issues.
Parts:
- removed FTDI: (no value), SparkFun-Connectors:1X06_NO_SILK
- removed JP2: (no value), SparkFun-Connectors:1X01
- added U$1: 1X7, headers(2mm):1X7
Connections:
- net !RESET: now also U$1.7; no longer JP2.1
- net DTR: now also U$1.6; no longer FTDI.1
- net GND: now also U$1.1, U$1.2; no longer FTDI.5, FTDI.6
- net RXO: now also U$1.5; no longer FTDI.2
- net TXO: now also U$1.4; no longer FTDI.3
- net VCC: now also U$1.3; no longer FTDI.4
Routing:
- net VCC: track 31.0 -> 32.9 mm
Changed lines of the file:
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@@
 </autorouter>
 <elements>
-<element name="FTDI" library="SparkFun-Connectors" package="1X06_NO_SILK" value="" x="12.9794" y="17.8562" rot="MR180">
-<attribute name="PROD_ID" value="CONN-08437" x="12.9794" y="17.8562" size="1.778" layer="28" rot="MR180" display="off"/>
-</element>
 <element name="SPI" library="SparkFun-Connectors" package="JST-4-PTH-VERT" value="" x="20.0914" y="1.651"/>
 <element name="FRAME1" library="SparkFun-Aesthetics" package="CREATIVE_COMMONS" value="FRAME-LETTER" x="14.3764" y="-8.1534"/>
 <element name="TX1" library="SparkFun-Connectors" package="JST-2-PTH-VERT" value="TX" x="14.1478" y="1.651"/>
-<element name="JP2" library="SparkFun-Connectors" package="1X01" value="" x="10.287" y="17.8308"/>
 <element name="JP1" library="SparkFun-Connectors" package="2X5_NOSILK" value="" x="2.3876" y="9.8044"/>
 <element name="JP3" library="SparkFun-Connectors" package="2X5_NOSILK" value="" x="7.4676" y="9.8044"/>
@@
 <element name="SPI1" library="SparkFun-Connectors" package="JST-4-PTH-VERT" value="" x="31.9532" y="1.651" rot="MR0"/>
 <element name="TX2" library="SparkFun-Connectors" package="JST-2-PTH-VERT" value="TX" x="37.8968" y="1.651" rot="MR0"/>
+<element name="U$1" library="headers(2mm)" package="1X7" value="1X7" x="16.2814" y="17.8308" rot="R180"/>
 </elements>
 <signals>
 <signal name="GND">
-<contactref element="FTDI" pad="6"/>
-<contactref element="FTDI" pad="5"/>
 <polygon width="0.4064" layer="1">
 <vertex x="-0.4064" y="19.2278"/>
@@
 <contactref element="JP1" pad="5"/>
 <contactref element="JP1" pad="7"/>
+<contactref element="U$1" pad="1"/>
+<contactref element="U$1" pad="2"/>
 </signal>
 <signal name="VCC">
-<contactref element="FTDI" pad="4"/>
 <contactref element="JP10" pad="2"/>
 <contactref element="JP10" pad="10"/>
@@
 <contactref element="JP10" pad="6"/>
 <contactref element="JP10" pad="8"/>
-<wire x1="20.5994" y1="17.8562" x2="20.5994" y2="17.145" width="0.4064" layer="16"/>
-<wire x1="20.5994" y1="17.145" x2="21.2852" y2="16.4592" width="0.4064" layer="16"/>
-<wire x1="21.2852" y1="16.4592" x2="38.5064" y2="16.4592" width="0.4064" layer="16"/>
+<wire x1="19.653" y1="16.4592" x2="38.5064" y2="16.4592" width="0.4064" layer="16"/>
 <wire x1="38.5064" y1="16.4592" x2="39.2684" y2="15.6972" width="0.4064" layer="16"/>
 <wire x1="39.2684" y1="15.6972" x2="39.2684" y2="15.0114" width="0.4064" layer="16"/>
@@
 <wire x1="39.2176" y1="9.8044" x2="39.2176" y2="7.2644" width="0.4064" layer="16"/>
 <wire x1="39.2176" y1="7.2644" x2="39.2176" y2="4.7244" width="0.4064" layer="16"/>
+<contactref element="U$1" pad="3"/>
+<wire x1="19.653" y1="16.4592" x2="18.2814" y2="17.8308" width="0.4064" layer="16"/>
 </signal>
 <signal name="DTR">
-<contactref element="FTDI" pad="1"/>
+<contactref element="U$1" pad="6"/>
 </signal>
 <signal name="RXO">
-<contactref element="FTDI" pad="2"/>
+<contactref element="U$1" pad="5"/>
 </signal>
 <signal name="TXO">
-<contactref element="FTDI" pad="3"/>
+<contactref element="U$1" pad="4"/>
 </signal>
 <signal name="MISO">
@@
 </signal>
 <signal name="!RESET">
-<contactref element="JP2" pad="1"/>
+<contactref element="U$1" pad="7"/>
 </signal>
 </signals>
