File: Tracksoar/tracksoar programmer.brd (EAGLE design)
At the start: 43.7 x 19.6 mm, 12 parts, among them U1 FT232RL-BASICSSOP

Commit message: replace headers
replaced 2.54mm headers on all production boards with 2mm headers to
resolve daughter board issues.
Parts:
- removed FTDI: (no value), SparkFun-Connectors:1X06_NO_SILK
- removed JP2: (no value), SparkFun-Connectors:1X01
- added U$1: 1X7, headers(2mm):1X7
Connections:
- net !RESET: now also U$1.7; no longer JP2.1
- net DTR: now also U$1.6, U1.2; no longer FTDI.1
- net GND: now also U$1.1, U$1.2; no longer FTDI.5, FTDI.6, U1.2
- net RXO: now also U$1.5; no longer FTDI.2
- net TXO: now also U$1.4; no longer FTDI.3
- net VCC: now also U$1.3; no longer FTDI.4
Routing:
- net DTR: track 0.00 -> 11.8 mm, vias 0 -> 1
- net RXO: track 26.0 -> 24.6 mm
- net TXO: track 16.1 -> 17.3 mm
Changed lines of the file:
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@@
 </autorouter>
 <elements>
-<element name="FTDI" library="SparkFun-Connectors" package="1X06_NO_SILK" value="" x="12.9794" y="17.8562" smashed="yes" rot="MR180">
-<attribute name="PROD_ID" value="CONN-08437" x="12.9794" y="17.8562" size="1.778" layer="28" rot="MR180" display="off"/>
-<attribute name="NAME" x="28.321" y="16.129" size="1.27" layer="25" ratio="10" rot="R180"/>
-<attribute name="VALUE" x="11.7094" y="21.0312" size="1.27" layer="28" rot="MR180"/>
-</element>
 <element name="SPI" library="SparkFun-Connectors" package="JST-4-PTH-VERT" value="" x="20.0914" y="1.651"/>
 <element name="FRAME1" library="SparkFun-Aesthetics" package="CREATIVE_COMMONS" value="FRAME-LETTER" x="14.3764" y="-8.1534"/>
 <element name="TX1" library="SparkFun-Connectors" package="JST-2-PTH-VERT" value="TX" x="14.1478" y="1.651"/>
-<element name="JP2" library="SparkFun-Connectors" package="1X01" value="" x="10.287" y="17.8308"/>
 <element name="ICSP" library="SparkFun-Connectors" package="2X3" value="AVR_SPI_PRG_6PTH" x="1.4732" y="6.8834" smashed="yes" rot="MR90">
 <attribute name="NAME" x="5.9182" y="5.6134" size="1.27" layer="26" ratio="10" rot="MR90"/>
@@
 <attribute name="VALUE" x="13.8684" y="9.525" size="1.27" layer="27" rot="R90"/>
 </element>
+<element name="U$1" library="headers(2mm)" package="1X7" value="1X7" x="16.2814" y="17.8308" rot="R180"/>
 </elements>
 <signals>
 <signal name="GND">
-<contactref element="FTDI" pad="6"/>
-<contactref element="FTDI" pad="5"/>
 <polygon width="0.4064" layer="1">
 <vertex x="-0.4064" y="19.2278"/>
@@
 <contactref element="U1" pad="11"/>
 <contactref element="U1" pad="3"/>
-<contactref element="U1" pad="2"/>
 <contactref element="U1" pad="26"/>
 <contactref element="U1" pad="25"/>
@@
 <contactref element="JP3" pad="GND"/>
 <via x="12.573" y="6.7564" extent="1-16" drill="0.6"/>
-<wire x1="20.9948" y1="14.578" x2="19.0448" y2="14.578" width="0" layer="19" extent="1-1"/>
+<contactref element="U$1" pad="1"/>
+<contactref element="U$1" pad="2"/>
+<wire x1="19.0448" y1="14.578" x2="20.9948" y2="14.578" width="0" layer="19" extent="1-1"/>
 </signal>
 <signal name="VCC">
-<contactref element="FTDI" pad="4"/>
 <contactref element="ICSP" pad="2"/>
 <contactref element="U1" pad="20"/>
@@
 <wire x1="19.6948" y1="14.578" x2="19.6948" y2="9.3738" width="0.3048" layer="1"/>
 <wire x1="19.6948" y1="9.3738" x2="20.1676" y2="8.901" width="0.3048" layer="1"/>
-<wire x1="20.5994" y1="17.8562" x2="20.5994" y2="17.272" width="0.3048" layer="1"/>
-<wire x1="20.5994" y1="17.272" x2="19.7104" y2="16.383" width="0.3048" layer="1"/>
 <wire x1="19.7104" y1="16.383" x2="19.7104" y2="14.5936" width="0.3048" layer="1"/>
 <wire x1="19.7104" y1="14.5936" x2="19.6948" y2="14.578" width="0.3048" layer="1"/>
@@
 <wire x1="15.9004" y1="5.08" x2="5.8166" y2="5.08" width="0.3048" layer="1"/>
 <wire x1="5.8166" y1="5.08" x2="4.0132" y2="6.8834" width="0.3048" layer="1"/>
+<contactref element="U$1" pad="3"/>
+<wire x1="18.2814" y1="17.8308" x2="18.2814" y2="17.812" width="0.3048" layer="1"/>
+<wire x1="18.2814" y1="17.812" x2="19.7104" y2="16.383" width="0.3048" layer="1"/>
 </signal>
 <signal name="DTR">
-<contactref element="FTDI" pad="1"/>
+<contactref element="U$1" pad="6"/>
+<contactref element="U1" pad="2"/>
+<wire x1="15.1448" y1="7.266" x2="15.1448" y2="9.0868" width="0.3048" layer="1"/>
+<wire x1="15.1448" y1="9.0868" x2="14.4018" y2="9.8298" width="0.3048" layer="1"/>
+<via x="14.4018" y="9.8298" extent="1-16" drill="0.6"/>
+<wire x1="14.4018" y1="9.8298" x2="12.2814" y2="11.9502" width="0.3048" layer="16"/>
+<wire x1="12.2814" y1="11.9502" x2="12.2814" y2="17.8308" width="0.3048" layer="16"/>
 </signal>
 <signal name="RXO">
-<contactref element="FTDI" pad="2"/>
 <contactref element="U1" pad="1"/>
-<wire x1="15.5194" y1="17.8562" x2="15.5194" y2="16.4084" width="0.3048" layer="1"/>
-<wire x1="15.5194" y1="16.4084" x2="15.113" y2="16.002" width="0.3048" layer="1"/>
-<wire x1="15.113" y1="16.002" x2="9.398" y2="16.002" width="0.3048" layer="1"/>
 <wire x1="9.398" y1="16.002" x2="8.0264" y2="14.6304" width="0.3048" layer="1"/>
 <wire x1="8.0264" y1="14.6304" x2="8.0264" y2="6.4516" width="0.3048" layer="1"/>
@@
 <wire x1="14.5034" y1="6.0452" x2="14.5034" y2="7.2574" width="0.3048" layer="1"/>
 <wire x1="14.5034" y1="7.2574" x2="14.4948" y2="7.266" width="0.3048" layer="1"/>
+<contactref element="U$1" pad="5"/>
+<wire x1="9.398" y1="16.002" x2="13.6652" y2="16.002" width="0.3048" layer="1"/>
+<wire x1="13.6652" y1="16.002" x2="14.2748" y2="16.6116" width="0.3048" layer="1"/>
+<wire x1="14.2748" y1="16.6116" x2="14.2748" y2="17.8242" width="0.3048" layer="1"/>
+<wire x1="14.2748" y1="17.8242" x2="14.2814" y2="17.8308" width="0.3048" layer="1"/>
 </signal>
 <signal name="TXO">
-<contactref element="FTDI" pad="3"/>
 <contactref element="U1" pad="5"/>
 <wire x1="17.0948" y1="7.266" x2="17.0948" y2="5.689" width="0.3048" layer="1"/>
@@
 <wire x1="17.5006" y1="5.2832" x2="18.3642" y2="5.2832" width="0.3048" layer="16"/>
 <wire x1="18.3642" y1="5.2832" x2="18.796" y2="5.715" width="0.3048" layer="16"/>
-<wire x1="18.796" y1="5.715" x2="18.796" y2="15.9766" width="0.3048" layer="16"/>
-<wire x1="18.796" y1="15.9766" x2="18.0848" y2="16.6878" width="0.3048" layer="16"/>
-<wire x1="18.0848" y1="16.6878" x2="18.0848" y2="17.8308" width="0.3048" layer="16"/>
-<wire x1="18.0848" y1="17.8308" x2="18.0594" y2="17.8562" width="0.3048" layer="16"/>
+<wire x1="18.796" y1="5.715" x2="18.796" y2="16.1798" width="0.3048" layer="16"/>
+<contactref element="U$1" pad="4"/>
+<wire x1="18.796" y1="16.1798" x2="18.542" y2="16.4338" width="0.3048" layer="16"/>
+<wire x1="18.542" y1="16.4338" x2="17.6784" y2="16.4338" width="0.3048" layer="16"/>
+<wire x1="17.6784" y1="16.4338" x2="16.2814" y2="17.8308" width="0.3048" layer="16"/>
 </signal>
 <signal name="MISO">
@@
 </signal>
 <signal name="!RESET">
-<contactref element="JP2" pad="1"/>
 <contactref element="ICSP" pad="5"/>
-<wire x1="10.287" y1="17.8308" x2="2.9972" y2="17.8308" width="0.3048" layer="1"/>
 <wire x1="2.9972" y1="17.8308" x2="1.4732" y2="16.3322" width="0.3048" layer="1"/>
 <wire x1="1.4732" y1="16.3322" x2="1.4732" y2="11.9634" width="0.3048" layer="1"/>
+<contactref element="U$1" pad="7"/>
+<wire x1="2.9972" y1="17.8308" x2="10.2814" y2="17.8308" width="0.3048" layer="1"/>
 </signal>
 <signal name="TXLED">
